Commit message: The perception module(pcd/normals obtain) has been almost completed.

File: assets/object/catapult/catapult.urdf (robot description, URDF)
Before this commit: robot catapult, 3 links, 2 joints
Links:
- removed link catapult
- added link catapult_body, mass 20.40400; collision box size=0.03000 0.30000 0.03000; collision box size=0.03000 0.30000 0.03000
- link button: mass 0.05089 -> 0.01
- link catapult_arm: mass 1.08000 -> 0.05
Joints:
- joint button_slider: parent catapult -> catapult_body
- joint catapult_hinge: parent catapult -> catapult_body
